File: CubeSatPowerAnalyticsUnit.kicad_sch (KiCad schematic)
At the start: 17 parts, among them J1 Conn_01x05_Pin, Q1 2N7002, T1 V_In (3,3V), T2 V_Out, T3 GND, T4 UART

Commit message: Initial commit - KiCad project v1.2
Parts:
- removed INV1: 74LVC1GU04DRL, Package_TO_SOT_SMD:SOT-553, symbol 74xGxx:74LVC1GU04DRL
- removed R2: 4K7 Ohm, Resistor_SMD:R_0805_2012Metric_Pad1.20x1.40mm_HandSolder, symbol Device:R
- C1, C2, C3: Purchase (none) -> https://www.lcsc.com/product-detail/C49678.html?s_z=n_C49678
- D1: Purchase (none) -> https://www.lcsc.com/product-detail/C188548.html?s_z=n_C188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
- INA1: Purchase (none) -> https://www.lcsc.com/product-detail/C59135.html
- J1: Purchase (none) -> https://www.lcsc.com/product-image/C2883689.html
- MCU1: Purchase (none) -> https://www.lcsc.com/product-detail/C1341298.html
- Q1: Purchase (none) -> https://www.lcsc.com/product-detail/C332103.html
- R1: value 0,1 Ohm -> 50 mOhm; Purchase (none) -> https://www.lcsc.com/product-detail/C49164908.html
- R2: renamed from R3; Purchase (none) -> https://www.lcsc.com/product-detail/C2889523.html?s_z=n_C28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
- R3: renamed from R4; Purchase (none) -> https://www.lcsc.com/product-detail/C17414.html
Connections:
- net at MCU1.19 (PA9): now also Q1.1 (G)
Other:
- note removed: "Inverter"
- moved on the sheet: J1

Commit message: Update PCB design - KiCad project v1.3
Parts:
- C1, C2, C3: LCSC (none) -> C49678; Purchase https://www.lcsc.com/product-detail/C49678.html?s_z=n_C49678 -> (none)
- D1: LCSC (none) -> C188548; Purchase https://www.lcsc.com/product-detail/C188548.html?s_z=n_C188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 -> (none)
- INA1: LCSC (none) -> C59135; Purchase https://www.lcsc.com/product-detail/C59135.html -> (none)
- J1: LCSC (none) -> C2883689; Purchase https://www.lcsc.com/product-image/C2883689.html -> (none)
- MCU1: LCSC (none) -> C1341298; Purchase https://www.lcsc.com/product-detail/C1341298.html -> (none)
- Q1: LCSC (none) -> C332103; Purchase https://www.lcsc.com/product-detail/C332103.html -> (none)
- R1: LCSC (none) -> C49164908; Purchase https://www.lcsc.com/product-detail/C49164908.html -> (none)
- R2: LCSC (none) -> C2889523; Purchase https://www.lcsc.com/product-detail/C2889523.html?s_z=n_C28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 -> (none)
- R3: LCSC (none) -> C17414; Purchase https://www.lcsc.com/product-detail/C17414.html -> (none)
- T1, T2, T3, T4: footprint TestPoint:TestPoint_THTPad_3.0x3.0mm_Drill1.5mm -> TestPoint:TestPoint_Pad_3.0x3.0mm
Changed lines of the file:
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@@
 			)
 		)
-		(property "Purchase" "https://www.lcsc.com/product-detail/C49678.html?s_z=n_C49678"
+		(property "LCSC" "C49678"
 			(at 119.38 64.77 90)
 			(effects
@@
 			)
 		)
-		(property "Footprint" "TestPoint:TestPoint_THTPad_3.0x3.0mm_Drill1.5mm"
+		(property "Footprint" "TestPoint:TestPoint_Pad_3.0x3.0mm"
 			(at 68.58 91.44 0)
 			(effects
@@
 			)
 		)
-		(property "Purchase" "https://www.lcsc.com/product-detail/C59135.html"
+		(property "LCSC" "C59135"
 			(at 119.38 73.66 0)
 			(effects
@@
 			)
 		)
-		(property "Purchase" "https://www.lcsc.com/product-detail/C1341298.html"
+		(property "LCSC" "C1341298"
 			(at 181.61 99.06 0)
 			(effects
@@
 			)
 		)
-		(property "Purchase" "https://www.lcsc.com/product-detail/C49678.html?s_z=n_C49678"
+		(property "LCSC" "C49678"
 			(at 146.05 76.2 0)
 			(effects
@@
 			)
 		)
-		(property "Purchase" "https://www.lcsc.com/product-detail/C2889523.html?s_z=n_C2889523"
+		(property "LCSC" "C2889523"
 			(at 140.97 73.66 90)
 			(effects
@@
 			)
 		)
-		(property "Purchase" "https://www.lcsc.com/product-image/C2883689.html"
+		(property "LCSC" "C2883689"
 			(at 81.28 57.15 0)
 			(effects
@@
 			)
 		)
-		(property "Purchase" "https://www.lcsc.com/product-detail/C188548.html?s_z=n_C188548"
+		(property "LCSC" "C188548"
 			(at 153.67 111.76 90)
 			(effects
@@
 			)
 		)
-		(property "Purchase" "https://www.lcsc.com/product-detail/C17414.html"
+		(property "LCSC" "C17414"
 			(at 165.1 69.85 0)
 			(effects
@@
 			)
 		)
-		(property "Purchase" "https://www.lcsc.com/product-detail/C49678.html?s_z=n_C49678"
+		(property "LCSC" "C49678"
 			(at 186.69 69.85 90)
 			(effects
@@
 			)
 		)
-		(property "Footprint" "TestPoint:TestPoint_THTPad_3.0x3.0mm_Drill1.5mm"
+		(property "Footprint" "TestPoint:TestPoint_Pad_3.0x3.0mm"
 			(at 68.58 81.28 0)
 			(effects
@@
 			)
 		)
-		(property "Purchase" "https://www.lcsc.com/product-detail/C332103.html"
+		(property "LCSC" "C332103"
 			(at 143.51 114.3 90)
 			(effects
@@
 			)
 		)
-		(property "Footprint" "TestPoint:TestPoint_THTPad_3.0x3.0mm_Drill1.5mm"
+		(property "Footprint" "TestPoint:TestPoint_Pad_3.0x3.0mm"
 			(at 68.58 71.12 0)
 			(effects
@@
 			)
 		)
-		(property "Purchase" "https://www.lcsc.com/product-detail/C49164908.html"
+		(property "LCSC" "C49164908"
 			(at 90.17 76.2 0)
 			(effects
@@
 			)
 		)
-		(property "Footprint" "TestPoint:TestPoint_THTPad_3.0x3.0mm_Drill1.5mm"
+		(property "Footprint" "TestPoint:TestPoint_Pad_3.0x3.0mm"
 			(at 68.58 101.6 0)
 			(effects

Commit message: Generate fabrication files - KiCad project v1.4
Parts:
- C1, C2, C3, D1, J1, R2, R3, T1, T2, T3, T4: now left out of the parts list
- R1: value 50 mOhm -> 0.05 Ohm
Changed lines of the file:
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@@
 		(unit 1)
 		(exclude_from_sim no)
-		(in_bom yes)
-		(on_board yes)
+		(in_bom no)
+		(on_board no)
 		(dnp no)
 		(property "Reference" "C1"
@@
 		)
 		(property "LCSC" "C49678"
+			(at 119.38 64.77 90)
+			(effects
+				(font
+					(size 1.27 1.27)
+				)
+				(hide yes)
+			)
+		)
+		(property "Purchase" ""
 			(at 119.38 64.77 90)
 			(effects
@@
 		(unit 1)
 		(exclude_from_sim no)
-		(in_bom yes)
-		(on_board yes)
+		(in_bom no)
+		(on_board no)
 		(dnp no)
 		(fields_autoplaced yes)
@@
 			)
 		)
+		(property "Purchase" ""
+			(at 63.5 91.44 0)
+			(effects
+				(font
+					(size 1.27 1.27)
+				)
+				(hide yes)
+			)
+		)
 		(pin "1"
 		)
@@
 		)
 		(property "LCSC" "C59135"
+			(at 119.38 73.66 0)
+			(effects
+				(font
+					(size 1.27 1.27)
+				)
+				(hide yes)
+			)
+		)
+		(property "Purchase" ""
 			(at 119.38 73.66 0)
 			(effects
@@
 			)
 		)
+		(property "Purchase" ""
+			(at 181.61 99.06 0)
+			(effects
+				(font
+					(size 1.27 1.27)
+				)
+				(hide yes)
+			)
+		)
 		(pin "32"
 		)
@@
 		(unit 1)
 		(exclude_from_sim no)
-		(in_bom yes)
-		(on_board yes)
+		(in_bom no)
+		(on_board no)
 		(dnp no)
 		(property "Reference" "C2"
@@
 			)
 		)
+		(property "Purchase" ""
+			(at 146.05 76.2 0)
+			(effects
+				(font
+					(size 1.27 1.27)
+				)
+				(hide yes)
+			)
+		)
 		(pin "1"
 		)
@@
 		(unit 1)
 		(exclude_from_sim no)
-		(in_bom yes)
-		(on_board yes)
+		(in_bom no)
+		(on_board no)
 		(dnp no)
 		(property "Reference" "R2"
@@
 		)
 		(property "LCSC" "C2889523"
+			(at 140.97 73.66 90)
+			(effects
+				(font
+					(size 1.27 1.27)
+				)
+				(hide yes)
+			)
+		)
+		(property "Purchase" ""
 			(at 140.97 73.66 90)
 			(effects
@@
 		(unit 1)
 		(exclude_from_sim no)
-		(in_bom yes)
-		(on_board yes)
+		(in_bom no)
+		(on_board no)
 		(dnp no)
 		(fields_autoplaced yes)
@@
 			)
 		)
+		(property "Purchase" ""
+			(at 81.28 57.15 0)
+			(effects
+				(font
+					(size 1.27 1.27)
+				)
+				(hide yes)
+			)
+		)
 		(pin "1"
 		)
@@
 		(unit 1)
 		(exclude_from_sim no)
-		(in_bom yes)
-		(on_board yes)
+		(in_bom no)
+		(on_board no)
 		(dnp no)
 		(fields_autoplaced yes)
@@
 			)
 		)
+		(property "Purchase" ""
+			(at 153.67 111.76 90)
+			(effects
+				(font
+					(size 1.27 1.27)
+				)
+				(hide yes)
+			)
+		)
 		(pin "2"
 		)
@@
 		(unit 1)
 		(exclude_from_sim no)
-		(in_bom yes)
-		(on_board yes)
+		(in_bom no)
+		(on_board no)
 		(dnp no)
 		(property "Reference" "R3"
@@
 			)
 		)
+		(property "Purchase" ""
+			(at 165.1 69.85 0)
+			(effects
+				(font
+					(size 1.27 1.27)
+				)
+				(hide yes)
+			)
+		)
 		(pin "1"
 		)
@@
 		(unit 1)
 		(exclude_from_sim no)
-		(in_bom yes)
-		(on_board yes)
+		(in_bom no)
+		(on_board no)
 		(dnp no)
 		(property "Reference" "C3"
@@
 		)
 		(property "LCSC" "C49678"
+			(at 186.69 69.85 90)
+			(effects
+				(font
+					(size 1.27 1.27)
+				)
+				(hide yes)
+			)
+		)
+		(property "Purchase" ""
 			(at 186.69 69.85 90)
 			(effects
@@
 		(unit 1)
 		(exclude_from_sim no)
-		(in_bom yes)
-		(on_board yes)
+		(in_bom no)
+		(on_board no)
 		(dnp no)
 		(fields_autoplaced yes)
@@
 			)
 		)
+		(property "Purchase" ""
+			(at 63.5 81.28 0)
+			(effects
+				(font
+					(size 1.27 1.27)
+				)
+				(hide yes)
+			)
+		)
 		(pin "1"
 		)
@@
 			)
 		)
+		(property "Purchase" ""
+			(at 143.51 114.3 90)
+			(effects
+				(font
+					(size 1.27 1.27)
+				)
+				(hide yes)
+			)
+		)
 		(pin "1"
 		)
@@
 		(unit 1)
 		(exclude_from_sim no)
-		(in_bom yes)
-		(on_board yes)
+		(in_bom no)
+		(on_board no)
 		(dnp no)
 		(fields_autoplaced yes)
@@
 			)
 		)
+		(property "Purchase" ""
+			(at 63.5 71.12 0)
+			(effects
+				(font
+					(size 1.27 1.27)
+				)
+				(hide yes)
+			)
+		)
 		(pin "1"
 		)
@@
 			)
 		)
-		(property "Value" "50 mOhm"
+		(property "Value" "0.05 Ohm"
 			(at 91.948 76.962 0)
 			(effects
@@
 			)
 		)
+		(property "Purchase" ""
+			(at 90.17 76.2 0)
+			(effects
+				(font
+					(size 1.27 1.27)
+				)
+				(hide yes)
+			)
+		)
 		(pin "1"
 		)
@@
 		(unit 1)
 		(exclude_from_sim no)
-		(in_bom yes)
-		(on_board yes)
+		(in_bom no)
+		(on_board no)
 		(dnp no)
 		(fields_autoplaced yes)
@@
 			(at 63.5 101.6 0)
 			(effects
+				(font
+					(size 1.27 1.27)
+				)
+				(hide yes)
+			)
+		)
+		(property "Purchase" ""
+			(at 63.5 101.6 0)
+			(effects

Commit message: Modify various footprints - KiCad project v1.5
Parts:
- C1, C2, C3, J1, R2, R3, T1, T2, T3, T4: now in the parts list
- D1: footprint Diode_SMD:D_SOD-123 -> Diode_SMD:D_SOD-323_HandSoldering; now in the parts list
Changed lines of the file:
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@@
 		(unit 1)
 		(exclude_from_sim no)
-		(in_bom no)
-		(on_board no)
+		(in_bom yes)
+		(on_board yes)
 		(dnp no)
 		(property "Reference" "C1"
@@
 		(unit 1)
 		(exclude_from_sim no)
-		(in_bom no)
-		(on_board no)
+		(in_bom yes)
+		(on_board yes)
 		(dnp no)
 		(fields_autoplaced yes)
@@
 		(unit 1)
 		(exclude_from_sim no)
-		(in_bom no)
-		(on_board no)
+		(in_bom yes)
+		(on_board yes)
 		(dnp no)
 		(property "Reference" "C2"
@@
 		(unit 1)
 		(exclude_from_sim no)
-		(in_bom no)
-		(on_board no)
+		(in_bom yes)
+		(on_board yes)
 		(dnp no)
 		(property "Reference" "R2"
@@
 		(unit 1)
 		(exclude_from_sim no)
-		(in_bom no)
-		(on_board no)
+		(in_bom yes)
+		(on_board yes)
 		(dnp no)
 		(fields_autoplaced yes)
@@
 		(unit 1)
 		(exclude_from_sim no)
-		(in_bom no)
-		(on_board no)
+		(in_bom yes)
+		(on_board yes)
 		(dnp no)
 		(fields_autoplaced yes)
@@
 			)
 		)
-		(property "Footprint" "Diode_SMD:D_SOD-123"
+		(property "Footprint" "Diode_SMD:D_SOD-323_HandSoldering"
 			(at 149.225 111.76 0)
 			(effects
@@
 		(unit 1)
 		(exclude_from_sim no)
-		(in_bom no)
-		(on_board no)
+		(in_bom yes)
+		(on_board yes)
 		(dnp no)
 		(property "Reference" "R3"
@@
 		(unit 1)
 		(exclude_from_sim no)
-		(in_bom no)
-		(on_board no)
+		(in_bom yes)
+		(on_board yes)
 		(dnp no)
 		(property "Reference" "C3"
@@
 		(unit 1)
 		(exclude_from_sim no)
-		(in_bom no)
-		(on_board no)
+		(in_bom yes)
+		(on_board yes)
 		(dnp no)
 		(fields_autoplaced yes)
@@
 		(unit 1)
 		(exclude_from_sim no)
-		(in_bom no)
-		(on_board no)
+		(in_bom yes)
+		(on_board yes)
 		(dnp no)
 		(fields_autoplaced yes)
@@
 		(unit 1)
 		(exclude_from_sim no)
-		(in_bom no)
-		(on_board no)
+		(in_bom yes)
+		(on_board yes)
 		(dnp no)
 		(fields_autoplaced yes)
